Commit message: Camera attached and functional!!!

File: husky_customization/husky_custom_description/urdf/custom_description.urdf.xacro (robot description, xacro)
@@ -25,24 +25,34 @@
   <xacro:arg name="ur5_enabled" default="$(optenv HUSKY_UR5_ENABLED false)" />
   <xacro:arg name="kinect_enabled" default="false" />
-  <!-- <xacro:include filename="$(find husky_description)/urdf/husky.urdf.xacro" />
-  <xacro:husky_robot /> -->
+  <xacro:include filename="$(find husky_custom_gazebo)/urdf/custom_description.gazebo.xacro"/>
   <!-- Insert customization below, sample provided: -->
-  <link name="bowler_link">
-    <visual>
+  <xacro:property name="camera_prop" value="0.05" />
+  <joint name="camera_joint" type="fixed">
+    <parent link="top_plate_link"/>
+    <child link="left_camera_link"/>
+    <origin rpy="0 0 0" xyz="0.3 0.23 0.03"/>
+    <axis xyz="0 1 0"/>
+  </joint>
+  <link name="left_camera_link">
+    <collision>
+      <origin xyz="0 0 0" rpy="0 0 0"/>
       <geometry>
-        <mesh filename="package://husky_custom_description/meshes/red_bowler.dae" />
-      </geometry>
-    </visual>
-    <collision>
-      <origin xyz="0 0 0.07" rpy="0 0 0" />
-      <geometry>
-        <box size="0.32 0.25 0.14" rpy="0 0 0"/>
+        <box size="${camera_prop} ${camera_prop} ${camera_prop}"/>
       </geometry>
     </collision>
+    <visual>
+      <origin xyz="0 0 0" rpy="0 0 0"/>
+      <geometry>
+        <box size="${camera_prop} ${camera_prop} ${camera_prop}"/>
+      </geometry>
+      <pose frame=''>0 0 0 0 -0 0</pose>
+      <transparency>0</transparency>
+      <cast_shadows>1</cast_shadows>
+    </visual>
+    <inertial>
+      <mass value="0.001" />
+      <origin xyz="0 0 0" rpy="0 0 0" />
+      <inertia ixx="0.0001" ixy="0" ixz="0" iyy="0.0001" iyz="0" izz="0.0001" />
+    </inertial>
   </link>
-  <joint name="bowler_joint" type="fixed">
-    <parent link="top_plate_link" />
-    <child link="bowler_link" />
-    <origin xyz="0.1 -0.1 0" rpy="0 0 0.5" />
-  </joint>
 </robot>

File: husky_customization/husky_custom_gazebo/urdf/custom_description.gazebo.xacro (robot description, xacro)
@@ -25,13 +25,37 @@
   <xacro:arg name="ur5_enabled" default="false" />
   <xacro:arg name="kinect_enabled" default="false" />
-  <xacro:include filename="$(find husky_gazebo)/urdf/husky.gazebo.xacro" />
-  <!-- Gazebo plugin for ROS Control -->
-  <gazebo>
-    <plugin name="gazebo_ros_control" filename="libgazebo_ros_control.so">
-      <robotNamespace>/</robotNamespace>
-    </plugin>
-  </gazebo>
-  <xacro:husky_robot_gazebo />
-  <xacro:include filename="$(find husky_custom_description)/urdf/custom_description.urdf.xacro" />
-  <!-- Insert customizations below: -->
+  <!-- camera -->
+    <gazebo reference="left_camera_link">
+      <sensor type="camera" name="camera_left">
+        <update_rate>30</update_rate>
+        <camera name='head'>
+        <horizontal_fov>1.047</horizontal_fov>
+          <image>
+            <width>320</width>
+            <height>240</height>
+            <format>R8G8B8</format>
+          </image>
+          <clip>
+            <near>0.02</near>
+            <far>300</far>
+          </clip>
+        </camera>
+        <always_on>1</always_on>
+        <visualize>1</visualize>
+        <plugin name="camera_controller" filename="libgazebo_ros_camera.so">
+          <alwaysOn>true</alwaysOn>
+          <updateRate>0.0</updateRate>
+          <cameraName>sensor/camera</cameraName>
+          <imageTopicName>image_raw</imageTopicName>
+          <cameraInfoTopicName>camera_info</cameraInfoTopicName>
+          <frameName>camera_link_optical</frameName>
+          <hackBaseline>0.07</hackBaseline>
+          <distortionK1>0.0</distortionK1>
+          <distortionK2>0.0</distortionK2>
+          <distortionK3>0.0</distortionK3>
+          <distortionT1>0.0</distortionT1>
+          <distortionT2>0.0</distortionT2>
+        </plugin>
+      </sensor>
+    </gazebo>
 </robot>

Commit message: Updates camera position

File: husky_customization/husky_custom_description/urdf/custom_description.urdf.xacro (robot description, xacro)
@@ -31,6 +31,6 @@
     <parent link="top_plate_link"/>
     <child link="left_camera_link"/>
-    <origin rpy="0 0 0" xyz="0.3 0.23 0.03"/>
-    <axis xyz="0 1 0"/>
+    <origin rpy="0 0 0" xyz="0.32 0.2 0.03"/>
+    <axis xyz="0 0 0"/>
   </joint>
   <link name="left_camera_link">
